File: ESP8285 PlantLight.kicad_sch (KiCad schematic)
At the start: 31 parts, among them U1 ESP8285, Y1 26Mhz

Commit message: space session
Parts:
- C1: value C_Small -> 10uF
- R1, R2, R3, R6: value R_Small -> 10K
Connections:
- net VDD3V3: no longer R1.1, R3.1, R4.1, R6.1
- new net +3V3: R1.1, R3.1, R4.1, R6.1

Commit message: sat session
Parts:
- added AE1: Antenna, RF_Antenna:Texas_SWRA117D_2.4GHz_Right, symbol Device:Antenna_Shield
- C1: footprint (none) -> Capacitor_SMD:C_0603_1608Metric
- C2, C4: value C_Small -> 100nF; footprint (none) -> Capacitor_SMD:C_0603_1608Metric
- C3: value C_Small -> 2.4pF; footprint (none) -> Capacitor_SMD:C_0603_1608Metric
- C7: value C_Small -> 1uF; footprint (none) -> Capacitor_SMD:C_0603_1608Metric
- C8: value C_Small -> 3.0pF; footprint (none) -> Capacitor_SMD:C_0603_1608Metric
- C9: value C_Small -> 10nF; footprint (none) -> Capacitor_SMD:C_0603_1608Metric
- L1: value L_Small -> 2.2nH; footprint (none) -> Inductor_SMD:L_0603_1608Metric
- R1, R2, R3, R6: footprint (none) -> Resistor_SMD:R_0603_1608Metric
- R4: value R_Small -> 10k; footprint (none) -> Resistor_SMD:R_0603_1608Metric
Connections:
- net GND: now also AE1.2 (Shield)
- net at C8.1, L1.2: now also AE1.1 (A)

Commit message: mon session
Parts:
- added C11: 1uF, Capacitor_SMD:C_0603_1608Metric, symbol Device:C_Small
- added C12: 100nF, symbol Device:C_Small
- added C13: 1uF, symbol Device:C_Small
- added D1: 3v3 Zener, Package_TO_SOT_SMD:SOT-23, symbol Diode:BZX84Cxx
- added FB1: 100R, Resistor_SMD:R_0603_1608Metric, symbol Device:FerriteBead
- added J1, J2: Screw_Terminal_01x01, Library:Keystone_16mm_19mm_18650, symbol Connector:Screw_Terminal_01x01
- added Q1: P-Chan Mosfet, Package_SON:Diodes_PowerDI3333-8, symbol Transistor_FET:DMP3013SFV
- added R7: 10K, symbol Device:R_Small
- added R8: 10K, Resistor_SMD:R_0603_1608Metric, symbol Device:R_Small
- added U2: RT9193-33GB, SOT94P279X129-5N, symbol RT9193-33GB:RT9193-33GB
- AE1: footprint RF_Antenna:Texas_SWRA117D_2.4GHz_Right -> RF_Antenna:Johanson_2450AT43F0100; symbol Device:Antenna_Shield -> Device:Antenna
- C10: value C_Small -> 100nF
- C5, C6: footprint Capacitor_SMD:C_0603_1608Metric -> Capacitor_SMD:C_01005_0402Metric
- renumbered GPIO15 to GPIO1, GPIO0 to GPIO3, GPIO13 to GPIO4, GPIO12 to GPIO5, GPIO14 to GPIO6, GPIO4 to GPIO7, GPIO5 to GPIO8
Connections:
- net GND renamed -BATT
- net -BATT: now also C11.1, C12.1, C13.1, D1.3 (K), J1.1 (Pin_1), U2.2 (GND); no longer AE1.2 (Shield)
- new net: C11.2, C12.2, FB1.2, R7.1, U2.1 (VIN)
- new net: R7.2, U2.3 (EN)
- new net: Q1.4 (G), R8.1
- new net: D1.1 (A), R8.2
- new net +3.3V: C13.2, U2.5 (VOUT)
- new net +BATT: J2.1 (Pin_1), Q1.5 (D)
- new net V_Bat: FB1.1, Q1.1 (S), Q1.2 (S), Q1.3 (S)
- no-connect marks 7 -> 8
Other:
- moved on the sheet: R2, R3, R4

Commit message: sat session
Parts:
- removed J1, J2: Screw_Terminal_01x01, Library:Keystone_16mm_19mm_18650, symbol Connector:Screw_Terminal_01x01
- added BT1: 18650, Library:18650_footprint, symbol Device:Battery_Cell
- added C14, C15, C16, C17: 100nF, Capacitor_SMD:C_0402_1005Metric, symbol Device:C_Small
- added D2, D3, D4, D5: WS2812B, LED_SMD:LED_WS2812B_PLCC4_5.0x5.0mm_P3.2mm, symbol LED:WS2812B
- added J1: Conn_01x03_Female, Connector_PinHeader_2.54mm:PinHeader_1x03_P2.54mm_Vertical, symbol Connector:Conn_01x03_Female
- added R10: 1M, Capacitor_SMD:C_0402_1005Metric, symbol Device:R_Small
- added R11: 300K, symbol Device:R_Small
- added R12, R13, R9: 330, Capacitor_SMD:C_0402_1005Metric, symbol Device:R_Small
- added U3, U4: SFH617A-1X007T, Package_DIP:SMDIP-4_W9.53mm_Clearance8mm, symbol Isolator:SFH617A-1X007T
- C12: footprint (none) -> Capacitor_SMD:C_0402_1005Metric
- C2, C4: footprint Capacitor_SMD:C_0603_1608Metric -> Capacitor_SMD:C_0402_1005Metric
- C5, C6: value 12pF -> 10pF
Connections:
- net +BATT: now also BT1.1 (+), J1.3 (Pin_3)
- net -BATT: now also BT1.2 (-), C14.2, C15.2, C16.2, C17.2, D2.3 (VSS), D3.3 (VSS), D4.3 (VSS), D5.3 (VSS), J1.2 (Pin_2), R11.1, R13.2
- net ADC: now also U3.3, U4.3
- net GPIO4: now also D2.4 (DIN)
- net GPIO5: now also R9.1
- net LNA: now reaches C3.1, L1.1, U1.2 (LNA)
- new net: R12.2, U4.1
- new net: R9.2, U3.1, U4.2
- new net: R10.1, R11.2, U4.4
- new net: R13.1, U3.2
- new net: D3.2 (DOUT), D4.4 (DIN)
- new net: D2.2 (DOUT), D3.4 (DIN)
- new net: J1.1 (Pin_1), U3.4
- new net: D4.2 (DOUT), D5.4 (DIN)
- new net V_BAT: C14.1, C15.1, C16.1, C17.1, D2.1 (VDD), D3.1 (VDD), D4.1 (VDD), D5.1 (VDD), R10.2, R12.1
- no-connect marks 8 -> 10
Other:
- moved on the sheet: 3.3V1, AE1, C1, C10, C11, C12, C13, C2, C3, C4, C5, C6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

Commit message: sun session
Parts:
- removed GPIO1, GPIO2, GPIO4, GPIO5, GPIO6, GPIO7, GPIO8: TestPoint_Small, TestPoint:TestPoint_Pad_D1.0mm, symbol Connector:TestPoint_Small
- removed U3, U4: SFH617A-1X007T, Package_DIP:SMDIP-4_W9.53mm_Clearance8mm, symbol Isolator:SFH617A-1X007T
- added U3, U4: TLP185, Package_SO:SOIC-4_4.55x3.7mm_P2.54mm, symbol Isolator:TLP185
- AE1: symbol Device:Antenna -> Device:Antenna_Chip
- C10: footprint (none) -> Capacitor_SMD:C_0402_1005Metric
- C13: footprint (none) -> Capacitor_SMD:C_0603_1608Metric
- C3, C8: footprint Capacitor_SMD:C_0603_1608Metric -> Capacitor_SMD:C_01005_0402Metric
- C9: footprint Capacitor_SMD:C_0603_1608Metric -> Capacitor_SMD:C_0402_1005Metric
- J1: value Conn_01x03_Female -> 01x03
- L1: footprint Inductor_SMD:L_0603_1608Metric -> Inductor_SMD:L_01005_0402Metric
- Q1: footprint Package_SON:Diodes_PowerDI3333-8 -> Package_SON:VSON-8_3.3x3.3mm_P0.65mm_NexFET
- R1: footprint Resistor_SMD:R_0603_1608Metric -> Resistor_SMD:R_01005_0402Metric
- R11, R7: footprint (none) -> Resistor_SMD:R_0402_1005Metric
- R2, R3, R4, R5, R6, R8: footprint Resistor_SMD:R_0603_1608Metric -> Resistor_SMD:R_0402_1005Metric
- renumbered GPIO3 to GPIO0
Connections:
- net +3V3 is gone; now on net 3V3: R1.1, R3.1, R4.1, R6.1
- net VDD3V3 is gone; now on net 3V3: 3.3V1.1, C10.1, C2.2, C4.2, C7.2, C9.1, U1.1 (VDDA), U1.11 (VDDPST), U1.17 (VDDPST), U1.29 (VDDD), U1.3 (VDD3P3), U1.30 (VDDA), U1.4 (VDD3P3)
- net V_Bat is gone; now on net V_BAT: FB1.1, Q1.1 (S), Q1.2 (S), Q1.3 (S)
- net ADC: now also U3.4, U4.4
- net V_BAT: now also J1.2 (Pin_2)
- net at R12.2: now also U3.1
- net at R9.2: now also U3.3, U4.1
- net at R10.1, R11.2: now also U3.6
- net at R13.1: now also U4.3
- net J1_ADC_IN: now reaches J1.1 (Pin_1)
- net J1_ADC_IN: now also U4.6
- net +3.3V renamed 3V3
- net +BATT renamed +BAT
- net +BAT: no longer J1.3 (Pin_3)
- net -BATT renamed GND
- net GND: now also J1.3 (Pin_3); no longer J1.2 (Pin_2)
Other:
- moved on the sheet: 3.3V1, C14, C15, C16, C17, C9, D2, D3, D4, D5, GND1, GPIO0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

Commit message: mon
Connections:
- net +BAT: now also Q1.1 (S), Q1.2 (S), Q1.3 (S); no longer Q1.5 (D)
- net GND: now also D1.1 (A); no longer D1.3 (K)
- net V_BAT: now also Q1.5 (D); no longer Q1.1 (S), Q1.2 (S), Q1.3 (S)
- net at R8.2: now also D1.3 (K); no longer D1.1 (A)
Other:
- moved on the sheet: D1
Changed lines of the file:
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@@
     (pin "9")
   )
-  (symbol (lib_id "Diode:BZX84Cxx") (at 69.85 151.13 0) (unit 1)
+  (symbol (lib_id "Diode:BZX84Cxx") (at 69.85 151.13 180) (unit 1)
     (in_bom yes) (on_board yes) (fields_autoplaced)
     (property "Reference" "D1" (id 0) (at 69.85 144.78 0))
@@
     (pin "2")
   )
-  (symbol (lib_id "Transistor_FET:DMP3013SFV") (at 90.17 151.13 0) (unit 1)
-    (in_bom yes) (on_board yes) (fields_autoplaced)
-    (property "Reference" "Q1" (id 0) (at 96.52 149.8599 0)
-      (effects (font (size 1.27 1.27)) (justify left))
-    )
-    (property "Value" "P-Chan Mosfet" (id 1) (at 96.52 152.3999 0)
-      (effects (font (size 1.27 1.27)) (justify left))
-    )
-    (property "Footprint" "Package_SON:VSON-8_3.3x3.3mm_P0.65mm_NexFET" (id 2) (at 95.25 153.035 0)
+  (symbol (lib_id "Transistor_FET:DMP3013SFV") (at 90.17 151.13 0) (mirror x) (unit 1)
+    (in_bom yes) (on_board yes) (fields_autoplaced)
+    (property "Reference" "Q1" (id 0) (at 96.52 152.4001 0)
+      (effects (font (size 1.27 1.27)) (justify left))
+    )
+    (property "Value" "P-Chan Mosfet" (id 1) (at 96.52 149.8601 0)
+      (effects (font (size 1.27 1.27)) (justify left))
+    )
+    (property "Footprint" "Package_SON:VSON-8_3.3x3.3mm_P0.65mm_NexFET" (id 2) (at 95.25 149.225 0)
       (effects (font (size 1.27 1.27) italic) (justify left) hide)
     )

Commit message: mon
Parts:
- removed D1: 3v3 Zener, Package_TO_SOT_SMD:SOT-23, symbol Diode:BZX84Cxx
- added C3: 100nF, Capacitor_SMD:C_0402_1005Metric, symbol Device:C_Small
- added Q1: IRLML2060, Package_TO_SOT_SMD:SOT-23, symbol Transistor_FET:IRLML2060
- added R5: 330, Capacitor_SMD:C_0402_1005Metric, symbol Device:R_Small
- added R6: 1K, Resistor_SMD:R_0402_1005Metric, symbol Device:R_Small
- added R9: 100, Resistor_SMD:R_0402_1005Metric, symbol Device:R_Small
- added U1: DW01, SOT23-6, symbol DW01:DW01
- renumbered C11 to C1, C6 to C10, C14 to C11, C7 to C12, C8 to C13, C15 to C14, C9 to C15, C10 to C16, C16 to C17, C17 to C18, C12 to C2, C1 to C4, C13 to C5, C2 to C6, C3 to C7, C4 to C8, C5 to C9, D2 to D1, D3 to D2, D4 to D3, D5 to D4, GPIO0 to GPIO1, Q1 to Q2, R5 to R10, R6 to R11, R9 to R12, R12 to R13, R13 to R14, R10 to R15, R11 to R16, U1 to U3, U3 to U5
Connections:
- net +BAT: now also R9.2
- net GND: now also C3.2, Q1.2 (S), U1.6 (GND)
- net at R8.2: now also Q1.3 (D), R6.2
- new net: Q1.1 (G), R5.1
- new net: R5.2, U1.1 (0D)
- new net: R6.1, U1.2 (CS)
- new net: C3.1, R9.1, U1.5 (VCC)
- no-connect marks 10 -> 12
Other:
- moved on the sheet: BT1, C1, C2, C5, FB1, Q2, R7, R8, U2

Commit message: tue session
Parts:
- R12, R13, R14: value 330 -> 330R
- R5: value 330 -> 10K
- R9: value 100 -> 100R
Other:
- moved on the sheet: 3.3V1, BT1, C1, C11, C14, C17, C18, C2, C3, C5, D1, D2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
