File: ESP8285 PlantLight.kicad_sch (KiCad schematic)
At the start: 56 parts, among them J1 01x03, Q1 IRLML2060, Q2 P-Chan Mosfet, U1 DW01, U2 RT9193-33GB, U3 ESP8285, U4 TLP185, U5 TLP185, Y1 26Mhz

Commit message: wed session
Parts:
- removed R12, R13: 330R, Capacitor_SMD:C_0402_1005Metric, symbol Device:R_Small
- removed U4, U5: TLP185, Package_SO:SOIC-4_4.55x3.7mm_P2.54mm, symbol Isolator:TLP185
- added C19: 100nF, Capacitor_SMD:C_0402_1005Metric, symbol Device:C_Small
- added R15: 1M, Capacitor_SMD:C_0402_1005Metric, symbol Device:R_Small
- added U4: 74LVC1G3157, 74LVC1G3157:SOP95P275X110-6N, symbol 74xGxx:74LVC1G3157
- R14: value 330R -> 300K; footprint Capacitor_SMD:C_0402_1005Metric -> Resistor_SMD:R_0402_1005Metric
- renumbered C3 to C1, C14 to C11, C5 to C14, C17 to C16, C16 to C17, C4 to C2, C1 to C3, C2 to C4, C6 to C5, C11 to C6, R5 to R1, R11 to R10, R7 to R11, R15 to R12, R16 to R13, R1 to R2, R2 to R3, R3 to R4, R4 to R5, R8 to R7, R9 to R8, R10 to R9, U3 to U2, U2 to U3
Connections:
- net ADC: now also U4.4
- net GND: now also C19.2, U4.2 (GND)
- net GPIO14: now also U4.6
- net GPIO4: no longer D1.4 (DIN)
- net GPIO5: now also D1.4 (DIN)
- net J1_ADC_IN: now also R15.1
- net at R14.1: now also R15.2, U4.3
- net at R12.1, R13.2: now also U4.1
- net 3V3 renamed VCC
- net VCC: now also C19.1, U4.5 (VCC)
Other:
- moved on the sheet: J1
