File: ESP8285 PlantLight.kicad_pcb (KiCad board)
At the start: 2 copper layers, 16 parts, among them U1 ESP8285, Y1 26Mhz

Commit message: space session
Parts:
- added R5: 12K, Resistor_SMD:R_0603_1608Metric, F.Cu at (132.1, 40.6)
Connections:
- C5 pad 1: Net-(U1-Pad27) -> Net-(C5-Pad1)
- C6 pad 1: Net-(U1-Pad28) -> Net-(C6-Pad1)
- GPIO12 pad 1: GPIO12 -> /GPIO12
- GPIO13 pad 1: GPIO13 -> /GPIO13
- GPIO14 pad 1: GPIO14 -> /GPIO14
- Y1 pad 1: Net-(U1-Pad28) -> Net-(C6-Pad1)
- Y1 pad 3: Net-(U1-Pad27) -> Net-(C5-Pad1)
Changed lines of the file:
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@@
   (net 25 "GPIO13")
   (net 26 "GPIO14")
+  (net 27 "Net-(C5-Pad1)")
+  (net 28 "Net-(C6-Pad1)")
+  (net 29 "/GPIO12")
+  (net 30 "/GPIO13")
+  (net 31 "/GPIO14")
+  (net 32 "Net-(R5-Pad2)")
+  (footprint "Resistor_SMD:R_0603_1608Metric" (layer "F.Cu")
+    (at 132.08 40.64)
+    (descr "Resistor SMD 0603 (1608 Metric), square (rectangular) end terminal, IPC_7351 nominal, (Body size source: IPC-SM-782 page 72, https://www.pcb-3d.com/wordpress/wp-content/uploads/ipc-sm-782a_amendment_1_and_2.pdf), generated with kicad-footprint-generator")
+    (tags "resistor")
+    (property "Sheetfile" "ESP8285 PlantLight.kicad_sch")
+    (property "Sheetname" "")
+    (attr smd)
+    (fp_text reference "R5" (at 0 -1.43) (layer "F.SilkS")
+      (effects (font (size 1 1) (thickness 0.15)))
+    )
+    (fp_text value "12K" (at 0 1.43) (layer "F.Fab")
+      (effects (font (size 1 1) (thickness 0.15)))
+    )
+    (fp_text user "${REFERENCE}" (at 0 0) (layer "F.Fab")
+      (effects (font (size 0.4 0.4) (thickness 0.06)))
+    )
+    (fp_line (start -0.237258 0.5225) (end 0.237258 0.5225) (layer "F.SilkS") (width 0.12))
+    (fp_line (start -0.237258 -0.5225) (end 0.237258 -0.5225) (layer "F.SilkS") (width 0.12))
+    (fp_line (start -1.48 -0.73) (end 1.48 -0.73) (layer "F.CrtYd") (width 0.05))
+    (fp_line (start 1.48 0.73) (end -1.48 0.73) (layer "F.CrtYd") (width 0.05))
+    (fp_line (start -1.48 0.73) (end -1.48 -0.73) (layer "F.CrtYd") (width 0.05))
+    (fp_line (start 1.48 -0.73) (end 1.48 0.73) (layer "F.CrtYd") (width 0.05))
+    (fp_line (start 0.8 0.4125) (end -0.8 0.4125) (layer "F.Fab") (width 0.1))
+    (fp_line (start 0.8 -0.4125) (end 0.8 0.4125) (layer "F.Fab") (width 0.1))
+    (fp_line (start -0.8 -0.4125) (end 0.8 -0.4125) (layer "F.Fab") (width 0.1))
+    (fp_line (start -0.8 0.4125) (end -0.8 -0.4125) (layer "F.Fab") (width 0.1))
+    (pad "1" smd roundrect (at -0.825 0) (size 0.8 0.95) (layers "F.Cu" "F.Paste" "F.Mask") (roundrect_rratio 0.25)
+      (net 20 "GND") (pintype "passive"))
+    (pad "2" smd roundrect (at 0.825 0) (size 0.8 0.95) (layers "F.Cu" "F.Paste" "F.Mask") (roundrect_rratio 0.25)
+      (net 32 "Net-(R5-Pad2)") (pintype "passive"))
+    (model "${KICAD6_3DMODEL_DIR}/Resistor_SMD.3dshapes/R_0603_1608Metric.wrl"
+      (offset (xyz 0 0 0))
+      (scale (xyz 1 1 1))
+      (rotate (xyz 0 0 0))
+    )
+  )
   (footprint "TestPoint:TestPoint_Pad_D1.0mm" (layer "F.Cu")
     (at 132.08 55.88)
@@
     (fp_circle (center 0 0) (end 1 0) (layer "F.CrtYd") (width 0.05) (fill none))
     (pad "1" smd circle (at 0 0) (size 1 1) (layers "F.Cu" "F.Mask")
-      (net 26 "GPIO14") (pinfunction "1") (pintype "passive"))
+      (net 31 "/GPIO14") (pinfunction "1") (pintype "passive"))
   )
   (footprint "TestPoint:TestPoint_Pad_D1.0mm" (layer "F.Cu")
@@
     (fp_circle (center 0 0) (end 1 0) (layer "F.CrtYd") (width 0.05) (fill none))
     (pad "1" smd circle (at 0 0) (size 1 1) (layers "F.Cu" "F.Mask")
-      (net 25 "GPIO13") (pinfunction "1") (pintype "passive"))
+      (net 30 "/GPIO13") (pinfunction "1") (pintype "passive"))
   )
   (footprint "ESP8285 (1):QFN50P500X500X90-33N" (layer "F.Cu")
@@
     (fp_circle (center 0 0) (end 1 0) (layer "F.CrtYd") (width 0.05) (fill none))
     (pad "1" smd circle (at 0 0) (size 1 1) (layers "F.Cu" "F.Mask")
-      (net 24 "GPIO12") (pinfunction "1") (pintype "passive"))
+      (net 29 "/GPIO12") (pinfunction "1") (pintype "passive"))
   )
   (footprint "Capacitor_SMD:C_0603_1608Metric" (layer "F.Cu")
@@
     (fp_line (start 0.8 0.4) (end -0.8 0.4) (layer "F.Fab") (width 0.1))
     (pad "1" smd roundrect (at -0.775 0 90) (size 0.9 0.95) (layers "F.Cu" "F.Paste" "F.Mask") (roundrect_rratio 0.25)
-      (net 15 "Net-(U1-Pad28)") (pintype "passive"))
+      (net 28 "Net-(C6-Pad1)") (pintype "passive"))
     (pad "2" smd roundrect (at 0.775 0 90) (size 0.9 0.95) (layers "F.Cu" "F.Paste" "F.Mask") (roundrect_rratio 0.25)
       (net 20 "GND") (pintype "passive"))
@@
     (fp_line (start 0.8 -0.4) (end 0.8 0.4) (layer "F.Fab") (width 0.1))
     (pad "1" smd roundrect (at -0.775 0 270) (size 0.9 0.95) (layers "F.Cu" "F.Paste" "F.Mask") (roundrect_rratio 0.25)
-      (net 14 "Net-(U1-Pad27)") (pintype "passive"))
+      (net 27 "Net-(C5-Pad1)") (pintype "passive"))
     (pad "2" smd roundrect (at 0.775 0 270) (size 0.9 0.95) (layers "F.Cu" "F.Paste" "F.Mask") (roundrect_rratio 0.25)
       (net 20 "GND") (pintype "passive"))
@@
     (fp_line (start 1.6 1.25) (end 1.6 -1.25) (layer "F.Fab") (width 0.1))
     (pad "1" smd rect (at -1.1 0.85) (size 1.4 1.2) (layers "F.Cu" "F.Paste" "F.Mask")
-      (net 15 "Net-(U1-Pad28)") (pinfunction "1") (pintype "passive"))
+      (net 28 "Net-(C6-Pad1)") (pinfunction "1") (pintype "passive"))
     (pad "2" smd rect (at 1.1 0.85) (size 1.4 1.2) (layers "F.Cu" "F.Paste" "F.Mask")
       (net 20 "GND") (pinfunction "2") (pintype "passive"))
     (pad "3" smd rect (at 1.1 -0.85) (size 1.4 1.2) (layers "F.Cu" "F.Paste" "F.Mask")
-      (net 14 "Net-(U1-Pad27)") (pinfunction "3") (pintype "passive"))
+      (net 27 "Net-(C5-Pad1)") (pinfunction "3") (pintype "passive"))
     (pad "4" smd rect (at -1.1 -0.85) (size 1.4 1.2) (layers "F.Cu" "F.Paste" "F.Mask")
       (net 20 "GND") (pinfunction "4") (pintype "passive"))

Commit message: sat session
Parts:
- added AE1: Antenna, RF_Antenna:Texas_SWRA117D_2.4GHz_Right, F.Cu at (131.7, 46.7)
- added C1: 10uF, Capacitor_SMD:C_0603_1608Metric, F.Cu at (111.0, 37.7)
- added C2: 100nF, Capacitor_SMD:C_0603_1608Metric, F.Cu at (137.7, 44.4)
- added C3: 2.4pF, Capacitor_SMD:C_0603_1608Metric, F.Cu at (137.7, 47.5)
- added C4: 100nF, Capacitor_SMD:C_0603_1608Metric, F.Cu at (136.1, 44.5)
- added C7: 1uF, Capacitor_SMD:C_0603_1608Metric, F.Cu at (136.9, 42.2)
- added C8: 3.0pF, Capacitor_SMD:C_0603_1608Metric, F.Cu at (133.1, 47.5)
- added C9: 10nF, Capacitor_SMD:C_0603_1608Metric, F.Cu at (134.6, 44.5)
- added L1: 2.2nH, Inductor_SMD:L_0603_1608Metric, F.Cu at (135.4, 46.7)
- added R1: 10K, Resistor_SMD:R_0603_1608Metric, F.Cu at (136.4, 37.1)
- added R2: 10K, Resistor_SMD:R_0603_1608Metric, F.Cu at (115.1, 37.7)
- added R3: 10K, Resistor_SMD:R_0603_1608Metric, F.Cu at (115.1, 35.2)
- added R4: 10k, Resistor_SMD:R_0603_1608Metric, F.Cu at (142.5, 55.6)
- added R6: 10K, Resistor_SMD:R_0603_1608Metric, F.Cu at (136.9, 49.8)
- moved 3.3V1 9.92 mm to (127.5, 65.8)
- moved GND1 9.92 mm to (130.0, 65.8)
- moved GPIO0 9.92 mm to (145.3, 65.8)
- moved GPIO13 9.92 mm to (137.7, 65.8)
- moved GPIO15 9.92 mm to (140.2, 65.8)
- moved GPIO4 9.92 mm to (147.8, 65.8)
- moved RX1 9.92 mm to (155.4, 65.8)
- moved GPIO12 9.92 mm to (135.1, 65.8)
- moved GPIO14 9.92 mm to (132.6, 65.8)
- moved GPIO2 9.92 mm to (142.7, 65.8)
- moved GPIO5 9.92 mm to (150.4, 65.8)
- moved TX1 9.92 mm to (152.9, 65.8)
- moved R5 7.91 mm to (140.0, 39.9)
- moved C6 2.70 mm to (139.2, 42.4)
- moved C5 2.70 mm to (145.3, 42.4)
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Connections:
- net GPIO4 renamed /GPIO4
- net GPIO5 renamed /GPIO5
- C5 pad 1: Net-(C5-Pad1) -> Net-(U1-Pad27)
- C6 pad 1: Net-(C6-Pad1) -> Net-(U1-Pad28)
- U1 pad 10: GPIO12 -> /GPIO12
- U1 pad 12: GPIO13 -> /GPIO13
- U1 pad 31: Net-(U1-Pad31) -> Net-(R5-Pad2)
- U1 pad 9: GPIO14 -> /GPIO14
- Y1 pad 1: Net-(C6-Pad1) -> Net-(U1-Pad28)
- Y1 pad 3: Net-(C5-Pad1) -> Net-(U1-Pad27)

Commit message: mon session
Parts:
- added C11: 1uF, Capacitor_SMD:C_0603_1608Metric, F.Cu at (99.6, 48.0)
- added D1: 3v3 Zener, Package_TO_SOT_SMD:SOT-23, F.Cu at (93.4, 46.2)
- added FB1: 100R, Resistor_SMD:R_0603_1608Metric, F.Cu at (98.2, 52.0)
- added J1: Screw_Terminal_01x01, Library:Keystone_16mm_19mm_18650, F.Cu at (139.7, 102.9)
- added J2: Screw_Terminal_01x01, Library:Keystone_16mm_19mm_18650, F.Cu at (139.7, 25.4)
- added Q1: P-Chan Mosfet, Package_SON:Diodes_PowerDI3333-8, F.Cu at (120.7, 51.6)
- added R8: 10K, Resistor_SMD:R_0603_1608Metric, F.Cu at (93.0, 56.3)
- AE1: footprint RF_Antenna:Texas_SWRA117D_2.4GHz_Right -> RF_Antenna:Johanson_2450AT43F0100
- C5, C6: footprint Capacitor_SMD:C_0603_1608Metric -> Capacitor_SMD:C_01005_0402Metric
- moved R2 6.60 mm to (112.3, 43.7)
- moved R1 3.59 mm to (136.9, 40.6)
- moved AE1 3.26 mm to (130.6, 49.8), turned to -90 degrees
- moved C6 1.14 mm to (139.7, 43.4)
- moved C5 0.72 mm to (144.8, 41.9)
- moved R4 0.72 mm to (142.0, 55.1)
- moved Y1 0.25 mm to (142.2, 42.7)
- renumbered GPIO15 to GPIO1, GPIO0 to GPIO3, GPIO13 to GPIO4, GPIO12 to GPIO5, GPIO14 to GPIO6, GPIO4 to GPIO7, GPIO5 to GPIO8
Connections:
- net /GPIO0 renamed GPIO0
- net /GPIO12 renamed GPIO12
- net /GPIO13 renamed GPIO13
- net /GPIO14 renamed GPIO14
- net /GPIO15 renamed GPIO15
- net /GPIO2 renamed GPIO2
- net /GPIO4 renamed GPIO4
- net /GPIO5 renamed GPIO5
- AE1 pad 2: GND -> (no net)

Commit message: sat session
Parts:
- removed J2: Screw_Terminal_01x01, Library:Keystone_16mm_19mm_18650
- added BT1: 18650, Library:18650_footprint, F.Cu at (139.7, 33.0)
- added C12: 100nF, Capacitor_SMD:C_0402_1005Metric, F.Cu at (152.4, 35.6)
- added C14: 100nF, Capacitor_SMD:C_0402_1005Metric, F.Cu at (170.2, 35.6)
- added C15: 100nF, Capacitor_SMD:C_0402_1005Metric, F.Cu at (177.1, 35.5)
- added C16: 100nF, Capacitor_SMD:C_0402_1005Metric, F.Cu at (167.3, 37.5)
- added C17: 100nF, Capacitor_SMD:C_0402_1005Metric, F.Cu at (164.4, 37.5)
- added D2: WS2812B, LED_SMD:LED_WS2812B_PLCC4_5.0x5.0mm_P3.2mm, F.Cu at (188.3, 31.2)
- added D3: WS2812B, LED_SMD:LED_WS2812B_PLCC4_5.0x5.0mm_P3.2mm, F.Cu at (179.9, 24.6)
- added D4: WS2812B, LED_SMD:LED_WS2812B_PLCC4_5.0x5.0mm_P3.2mm, F.Cu at (179.9, 31.2)
- added D5: WS2812B, LED_SMD:LED_WS2812B_PLCC4_5.0x5.0mm_P3.2mm, F.Cu at (188.3, 24.6)
- added Q2: Q_NPN_BCE, Package_TO_SOT_SMD:SOT-23, F.Cu at (158.3, 32.4)
- added Q3: Q_PNP_BCE, Package_TO_SOT_SMD:SOT-23, F.Cu at (153.4, 32.4)
- added R10: 1M, Capacitor_SMD:C_0402_1005Metric, F.Cu at (155.3, 35.6)
- added R12: 330, Capacitor_SMD:C_0402_1005Metric, F.Cu at (167.3, 35.6)
- added R13: 330, Capacitor_SMD:C_0402_1005Metric, F.Cu at (164.4, 35.6)
- added R9: 330, Capacitor_SMD:C_0402_1005Metric, F.Cu at (158.1, 35.6)
- added U3: SFH617A-1X007T, Package_DIP:SMDIP-4_W9.53mm_Clearance8mm, F.Cu at (169.3, 31.2)
- added U4: SFH617A-1X007T, Package_DIP:SMDIP-4_W9.53mm_Clearance8mm, F.Cu at (169.3, 24.6)
- C2, C4: footprint Capacitor_SMD:C_0603_1608Metric -> Capacitor_SMD:C_0402_1005Metric
- C5, C6: value 12pF -> 10pF
- J1: value Screw_Terminal_01x01 -> Conn_01x03_Female; footprint Library:Keystone_16mm_19mm_18650 -> Connector_PinHeader_2.54mm:PinHeader_1x03_P2.54mm_Vertical
- moved J1 54.3 mm to (154.9, 50.8), turned to 0 degrees
Connections:
- C3 pad 1: Net-(C3-Pad1) -> /LNA
- C5 pad 1: Net-(U1-Pad27) -> Net-(C5-Pad1)
- J1 pad 1: GND -> Net-(J1-Pad1)
- L1 pad 1: Net-(C3-Pad1) -> /LNA
- Y1 pad 3: Net-(U1-Pad27) -> Net-(C5-Pad1)

Commit message: mon
Parts:
- removed GPIO1, GPIO2, GPIO3, GPIO4, GPIO5, GPIO6, GPIO7, GPIO8: TestPoint_Small, TestPoint:TestPoint_Pad_D1.0mm
- removed Q2: Q_NPN_BCE, Package_TO_SOT_SMD:SOT-23
- removed Q3: Q_PNP_BCE, Package_TO_SOT_SMD:SOT-23
- added C10: 100nF, Capacitor_SMD:C_0402_1005Metric, F.Cu at (150.6, 72.1)
- added C13: 1uF, Capacitor_SMD:C_0603_1608Metric, F.Cu at (153.7, 63.2)
- added GPIO0: TestPoint_Small, TestPoint:TestPoint_Pad_D1.0mm, F.Cu at (158.8, 78.7)
- added R11: 300K, Resistor_SMD:R_0402_1005Metric, F.Cu at (148.1, 89.1)
- added R7: 10K, Resistor_SMD:R_0402_1005Metric, F.Cu at (149.9, 65.8)
- added U2: RT9193-33GB, RT9193-33GB:SOT94P279X129-5N, F.Cu at (150.9, 63.5)
- C3, C8: footprint Capacitor_SMD:C_0603_1608Metric -> Capacitor_SMD:C_01005_0402Metric
- C9: footprint Capacitor_SMD:C_0603_1608Metric -> Capacitor_SMD:C_0402_1005Metric
- J1: value Conn_01x03_Female -> 01x03
- L1: footprint Inductor_SMD:L_0603_1608Metric -> Inductor_SMD:L_01005_0402Metric
- Q1: footprint Package_SON:Diodes_PowerDI3333-8 -> Package_SON:VSON-8_3.3x3.3mm_P0.65mm_NexFET
- R1: footprint Resistor_SMD:R_0603_1608Metric -> Resistor_SMD:R_01005_0402Metric
- R2, R3, R4, R5, R6, R8: footprint Resistor_SMD:R_0603_1608Metric -> Resistor_SMD:R_0402_1005Metric
- U3, U4: value SFH617A-1X007T -> TLP185; footprint Package_DIP:SMDIP-4_W9.53mm_Clearance8mm -> Package_SO:SOIC-4_4.55x3.7mm_P2.54mm
- moved D5 90.6 mm to (157.2, 109.7), turned to -90 degrees
- moved D4 84.9 mm to (147.6, 109.7), turned to 90 degrees
- moved C14 75.1 mm to (151.1, 108.2), turned to 90 degrees
- moved U4 72.4 mm to (149.4, 94.2)
- moved C17 71.5 mm to (153.7, 108.2), turned to -90 degrees
- moved U3 70.4 mm to (149.4, 98.8)
- moved R12 63.0 mm to (157.2, 97.8)
- moved R3 62.1 mm to (157.5, 80.5), turned to 90 degrees
- moved R13 61.1 mm to (157.2, 96.3)
- moved C1 61.1 mm to (154.2, 81.0), turned to -90 degrees
- moved R8 59.6 mm to (152.6, 57.9), turned to 90 degrees
- moved D1 57.7 mm to (150.0, 57.3)
- moved R2 56.8 mm to (155.4, 80.5), turned to 90 degrees
- moved R10 51.6 mm to (148.1, 86.6), turned to 90 degrees
- moved FB1 50.4 mm to (147.8, 61.0)
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Connections:
- net GPIO15 renamed /GPIO15
- net GPIO2 renamed /GPIO2
- 3.3V1 pad 1: VDD3V3 -> 3V3
- AE1 pad 2: (no net) -> unconnected-(AE1-Pad2)
- BT1 pad 1: +BATT -> /+BAT
- C14 pad 1: /V_BAT -> V_BAT
- C15 pad 1: /V_BAT -> V_BAT
- C16 pad 1: /V_BAT -> V_BAT
- C17 pad 1: /V_BAT -> V_BAT
- C2 pad 2: VDD3V3 -> 3V3
- C4 pad 2: VDD3V3 -> 3V3
- C7 pad 2: VDD3V3 -> 3V3
- C9 pad 1: VDD3V3 -> 3V3
- D1 pad 1: Net-(D1-Pad1) -> GND
- D1 pad 3: GND -> Net-(D1-Pad3)
- D2 pad 1: /V_BAT -> V_BAT
- D3 pad 1: /V_BAT -> V_BAT
- D4 pad 1: /V_BAT -> V_BAT
- D5 pad 1: /V_BAT -> V_BAT
- FB1 pad 1: /V_Bat -> V_BAT
- J1 pad 1: Net-(J1-Pad1) -> /J1_ADC_IN
- J1 pad 2: GND -> V_BAT
- J1 pad 3: +BATT -> GND
- Q1 pad 1: /V_Bat -> /+BAT
- Q1 pad 2: /V_Bat -> /+BAT
- Q1 pad 3: /V_Bat -> /+BAT
- Q1 pad 5: +BATT -> V_BAT
- R1 pad 1: +3V3 -> 3V3
- R10 pad 2: /V_BAT -> V_BAT
- R12 pad 1: /V_BAT -> V_BAT
- R3 pad 1: +3V3 -> 3V3
- R4 pad 1: +3V3 -> 3V3
- R6 pad 1: +3V3 -> 3V3
- R8 pad 2: Net-(D1-Pad1) -> Net-(D1-Pad3)
- U1 pad 1: VDD3V3 -> 3V3
- U1 pad 11: VDD3V3 -> 3V3
- U1 pad 17: VDD3V3 -> 3V3
- U1 pad 2: Net-(C3-Pad1) -> /LNA
- U1 pad 27: Net-(U1-Pad27) -> Net-(C5-Pad1)
- U1 pad 29: VDD3V3 -> 3V3
- U1 pad 3: VDD3V3 -> 3V3
- U1 pad 30: VDD3V3 -> 3V3
- U1 pad 4: VDD3V3 -> 3V3
- U3 pad 1: Net-(R9-Pad2) -> Net-(R12-Pad2)
- U3 pad 3: ADC -> Net-(R9-Pad2)
- U3 pad 4: Net-(J1-Pad1) -> ADC
- U4 pad 1: Net-(R12-Pad2) -> Net-(R9-Pad2)
- U4 pad 3: ADC -> Net-(R13-Pad1)
- U4 pad 4: Net-(R10-Pad1) -> ADC

Commit message: mon
Parts:
- removed the D1 at (150.0, 57.3)
- added C3: 100nF, Capacitor_SMD:C_0402_1005Metric, F.Cu at (146.8, 58.7)
- added Q1: IRLML2060, Package_TO_SOT_SMD:SOT-23, F.Cu at (149.1, 60.5)
- added R5: 330, Capacitor_SMD:C_0402_1005Metric, F.Cu at (151.4, 58.7)
- added R6: 1K, Resistor_SMD:R_0402_1005Metric, F.Cu at (151.4, 56.6)
- added R9: 100, Resistor_SMD:R_0402_1005Metric, F.Cu at (146.8, 56.6)
- added U1: DW01, DW01:SOT23-6, F.Cu at (149.1, 57.1)
- moved FB1 5.86 mm to (153.7, 60.5), turned to 180 degrees
- moved C1 4.60 mm to (151.6, 62.7)
- moved C5 4.60 mm to (158.2, 62.7)
- moved U2 4.60 mm to (155.4, 63.0)
- moved C2 4.60 mm to (152.9, 62.5)
- moved R7 4.60 mm to (154.4, 65.3)
- moved 3.3V1 2.51 mm to (158.8, 60.2)
- moved GND1 2.18 mm to (158.8, 65.3)
- moved R8 0.84 mm to (152.9, 58.7), turned to 180 degrees
- moved Q2 0.80 mm to (156.0, 57.7)
- renumbered C11 to C1, C6 to C10, C14 to C11, C7 to C12, C8 to C13, C15 to C14, C9 to C15, C10 to C16, C16 to C17, C17 to C18, C12 to C2, C1 to C4, C13 to C5, C2 to C6, C3 to C7, C4 to C8, C5 to C9, D2 to D1, D3 to D2, D4 to D3, D5 to D4, GPIO0 to GPIO1, Q1 to Q2, R5 to R10, R6 to R11, R9 to R12, R12 to R13, R13 to R14, R10 to R15, R11 to R16, U1 to U3, U3 to U5

Commit message: wed session
Parts:
- removed the R13 at (157.2, 97.8)
- removed U5: TLP185, Package_SO:SOIC-4_4.55x3.7mm_P2.54mm
- added C19: 100nF, Capacitor_SMD:C_0402_1005Metric, F.Cu at (147.6, 88.1)
- added R15: 1M, Capacitor_SMD:C_0402_1005Metric, F.Cu at (153.4, 86.4)
- R1: renamed from R5; value 330 -> 10K
- R12: value 330 -> 1M
- R14: value 330 -> 300K; footprint Capacitor_SMD:C_0402_1005Metric -> Resistor_SMD:R_0402_1005Metric
- R8: renamed from R9; value 100 -> 100R
- U4: value TLP185 -> 74LVC1G3157; footprint Package_SO:SOIC-4_4.55x3.7mm_P2.54mm -> 74LVC1G3157:SOP95P275X110-6N
- moved R14 11.5 mm to (151.4, 86.4), turned to 180 degrees
- moved R12 6.86 mm to (153.4, 90.9), turned to 0 degrees
- moved U4 5.62 mm to (150.4, 88.6), turned to 180 degrees
- moved R13 3.76 mm to (151.4, 90.9), turned to 0 degrees
- moved R10 0.51 mm to (151.6, 82.0)
- renumbered C3 to C1, C14 to C11, C5 to C14, C17 to C16, C16 to C17, C4 to C2, C1 to C3, C2 to C4, C6 to C5, C11 to C6, R11 to R10, R7 to R11, R15 to R12, R16 to R13, R1 to R2, R2 to R3, R3 to R4, R4 to R5, R8 to R7, R10 to R9, U3 to U2, U2 to U3
Connections:
- D1 pad 4: GPIO4 -> GPIO5
- R12 pad 1: Net-(R15-Pad1) -> Net-(R12-Pad1)
- R12 pad 1: GPIO5 -> Net-(R12-Pad1)
- R12 pad 2: Net-(R12-Pad2) -> V_BAT
- R13 pad 2: Net-(R15-Pad1) -> Net-(R12-Pad1)
- U4 pad 1: Net-(R12-Pad2) -> Net-(R12-Pad1)
- U4 pad 6: /J1_ADC_IN -> GPIO14
